File: DG Nova 1200 CPU.kicad_sch (KiCad schematic)
At the start: 207 parts, among them Q1 MPS3640, U1 74LS122, U10 74LS20, U100 045, U101 74LS04, U102 74LS179, U103 74LS179, U105 74LS179, U106 74LS179, U107 74LS179, U108 74LS179, U109 74LS00, U11 74LS03, U110 74LS20, U111 74LS10, U112 74LS51, U113 74LS114, U114 74LS51, U115 74LS179, U116 74LS157, U117 74LS181, U118 74LS00, U119 74LS170, U12 74LS00, U120 8264, U121 74LS157, U122 74LS179, U123 8225, U124 8225, U125 8264, U13 045, U14 74LS20, U15 74LS20, U16 74LS04, U17 74LS179, U18 74LS20, U19 74LS00, U2 74LS74, U20 74LS74, U21 74LS00, U22 74LS04, U23 74LS179, U24 74LS51, U25 74LS139, U26 74LS04, U27 74LS04, U28 74LS179, U29 74LS179, U3 74LS00, U30 82S23, U31 82S23, U32 74LS179, U33 74LS179, U34 045, U35 74LS10, U36 74LS00, U37 74LS179, U38 74LS179, U39 74LS179, U4 045, U40 74LS179, U41 045, U42 74LS179, U43 74H54, U44 74LS51, U45 74LS51, U46 74H54, U47 74H54, U48 045, U49 74LS03, U5 74LS04, U50 74LS10, U51 74LS139, U52 74LS139, U53 045, U54 74LS179, U55 74LS51, U56 74LS20, U57 74LS00, U58 045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

Commit message: Deep Dives
Parts:
- added J1, J3: Conn_02x40_Odd_Even, Forgotten Machines:Card_Edge_Entrex_Trapezoid 80, symbol Connector_Generic:Conn_02x40_Odd_Even
- added J2, J4: DG Nova Card-Edge 81-100, Forgotten Machines:Data General Nova Card-Edge 81-100, symbol ForgottenMachines:DG_Nova_Card-Edge_81-100
Connections:
- net +5V: now also J1.3 (Pin_3), J1.4 (Pin_4), J2.97 (Pin_18), J2.98 (Pin_17), J3.3 (Pin_3), J3.4 (Pin_4), J4.97 (Pin_18), J4.98 (Pin_17)
- net CLK FLOP: now also J3.48 (Pin_48)
- net CLR: now also J1.50 (Pin_50)
- net DATIA: now also J1.44 (Pin_44)
- net DATIB: now also J1.42 (Pin_42)
- net DATIC: now also J1.54 (Pin_54)
- net DATOA: now also J1.58 (Pin_58)
- net DATOB: now also J1.56 (Pin_56)
- net DATOC: now also J1.48 (Pin_48)
- net DCHI: now also J3.37 (Pin_37)
- net DCHO: now also J3.33 (Pin_33)
- net INHIBIT: now also J3.30 (Pin_30)
- net INTA: now also J1.40 (Pin_40)
- net IO PLS: now also J1.74 (Pin_74)
- net IO RST: now also J1.70 (Pin_70)
- net LOAD IR: now also J1.73 (Pin_73)
- net MB LOAD: now also J3.74 (Pin_74)
- net MEM OK: now also J1.9 (Pin_9)
- net OVFLO: now also J3.39 (Pin_39)
- net RESTART ENABLE: now also J1.32 (Pin_32)
- net STROBE: now also J3.20 (Pin_20)
- net STRT: now also J1.52 (Pin_52)
- net ~{CARRY}: now also J1.15 (Pin_15)
- net ~{CON DATA}: now also J1.28 (Pin_28)
- net ~{CON INST}: now also J1.22 (Pin_22)
- net ~{CONT+ISTP+MSTP}: now also J1.25 (Pin_25)
- net ~{DCHA}: now also J1.60 (Pin_60)
- net ~{DCHM0}: now also J3.17 (Pin_17)
- net ~{DCHM1}: now also J3.21 (Pin_21)
- net ~{DCHR}: now also J3.35 (Pin_35)
- net ~{DEFER}: now also J1.12 (Pin_12)
- net ~{DIV}: now also J2.91 (Pin_12)
- net ~{DRIVE IO}: now also J4.88 (Pin_7)
- net ~{DS0}: now also J1.72 (Pin_72)
- net ~{DS1}: now also J1.68 (Pin_68)
- net ~{DS2}: now also J1.66 (Pin_66)
- net ~{DS3}: now also J1.46 (Pin_46)
- net ~{DS4}: now also J1.62 (Pin_62)
- net ~{DS5}: now also J1.64 (Pin_64)
- net ~{EXEC}: now also J1.11 (Pin_11)
- net ~{EXT LOAD}: now also J1.47 (Pin_47), J3.49 (Pin_49)
- net ~{FETCH}: now also J1.13 (Pin_13), J1.49 (Pin_49)
- net ~{FORCE LOAD IR}: now also J2.85 (Pin_6)
- net ~{INH TRANS}: now also J3.45 (Pin_45)
- net ~{INTR}: now also J3.29 (Pin_29)
- net ~{ION}: now also J1.16 (Pin_16)
- net ~{ISTP}: now also J1.17 (Pin_17)
- net ~{LOAD AC}: now also J1.77 (Pin_77)
- net ~{MA LOAD}: now also J3.7 (Pin_7)
- net ~{MB CLEAR}: now also J4.86 (Pin_5)
- net ~{MBO0}: now also J3.79 (Pin_79)
- net ~{MBO10}: now also J3.8 (Pin_8)
- net ~{MBO11}: now also J3.5 (Pin_5)
- net ~{MBO12}: now also J1.39 (Pin_39)
- net ~{MBO13}: now also J1.37 (Pin_37)
- net ~{MBO14}: now also J1.43 (Pin_43)
- net ~{MBO15}: now also J1.41 (Pin_41)
- net ~{MBO1}: now also J3.77 (Pin_77)
- net ~{MBO2}: now also J3.44 (Pin_44)
- net ~{MBO3}: now also J3.43 (Pin_43)
- net ~{MBO4}: now also J3.42 (Pin_42)
- net ~{MBO5}: now also J3.32 (Pin_32)
- net ~{MBO6}: now also J3.16 (Pin_16)
- net ~{MBO7}: now also J3.14 (Pin_14)
- net ~{MBO8}: now also J3.12 (Pin_12)
- net ~{MBO9}: now also J3.9 (Pin_9)
- net ~{MD SEL1}: now also J2.87 (Pin_8)
- net ~{MEM0}: now also J3.71 (Pin_71)
- net ~{MEM10}: now also J1.45 (Pin_45)
- net ~{MEM11}: now also J1.51 (Pin_51)
- net ~{MEM12}: now also J1.36 (Pin_36)
- net ~{MEM13}: now also J1.35 (Pin_35)
- net ~{MEM14}: now also J3.76 (Pin_76)
- net ~{MEM15}: now also J3.18 (Pin_18)
- net ~{MEM1}: now also J3.70 (Pin_70)
- net ~{MEM2}: now also J3.47 (Pin_47)
- net ~{MEM3}: now also J3.68 (Pin_68)
- net ~{MEM4}: now also J3.28 (Pin_28)
- net ~{MEM5}: now also J3.26 (Pin_26)
- net ~{MEM6}: now also J3.22 (Pin_22)
- net ~{MEM7}: now also J3.24 (Pin_24)
- net ~{MEM8}: now also J1.55 (Pin_55)
- net ~{MEM9}: now also J1.53 (Pin_53)
- net ~{MSKO}: now also J1.38 (Pin_38)
- net ~{MSTP}: now also J1.20 (Pin_20)
- net ~{PL}: now also J1.19 (Pin_19)
- net ~{POWER FAIL}: now also J1.5 (Pin_5)
- net ~{READ IO}: now also J4.83 (Pin_4)
- net ~{READ1}: now also J4.87 (Pin_8)
- net ~{READ2}: now also J4.90 (Pin_9)
- net ~{RQENB}: now also J3.41 (Pin_41)
- net ~{RST}: now also J1.30 (Pin_30)
- net ~{RUN}: now also J1.14 (Pin_14)
- net ~{SELB}: now also J2.82 (Pin_1)
- net ~{SELD}: now also J1.80 (Pin_80)
- net ~{SHIFT0}: now also J4.94 (Pin_13)
- net ~{SHIFT1}: now also J4.96 (Pin_15)
- net ~{SHIFT2}: now also J4.93 (Pin_14)
- net ~{SHIFT3}: now also J4.91 (Pin_12)
- net ~{SKIP}: now also J3.69 (Pin_69)
- net ~{STOP}: now also J1.31 (Pin_31)
- net ~{TEST}: now also J2.92 (Pin_11)
- net ~{WAS JSR}: now also J2.89 (Pin_10)
- net WHOA renamed ~{WHOA}
- net ~{WHOA}: now also J3.6 (Pin_6)
- net ~{CON_RQ} renamed ~{CON RQ}
- net ~{CON RQ}: now also J1.27 (Pin_27)
- new net +5V OK: J1.8 (Pin_8)
- new net GND: J1.1 (Pin_1), J1.2 (Pin_2), J1.33 (Pin_33), J1.34 (Pin_34), J2.100 (Pin_19), J2.99 (Pin_20), J3.1 (Pin_1), J3.2 (Pin_2), J3.50 (Pin_50), J4.100 (Pin_19), J4.99 (Pin_20)
- new net ~{DATA0}: J3.62 (Pin_62)
- new net ~{DATA10}: J3.75 (Pin_75)
- new net ~{DATA11}: J3.58 (Pin_58)
- new net ~{DATA12}: J3.59 (Pin_59)
- new net ~{DATA13}: J3.64 (Pin_64)
- new net ~{DATA14}: J3.56 (Pin_56)
- new net ~{DATA15}: J3.66 (Pin_66)
- new net ~{DATA1}: J3.65 (Pin_65)
- new net ~{DATA2}: J4.82 (Pin_1)
- new net ~{DATA3}: J3.73 (Pin_73)
- new net ~{DATA4}: J3.61 (Pin_61)
- new net ~{DATA5}: J3.57 (Pin_57)
- new net ~{DATA6}: J4.95 (Pin_16)
- new net ~{DATA7}: J3.55 (Pin_55)
- new net ~{DATA8}: J3.60 (Pin_60)
- new net ~{DATA9}: J3.63 (Pin_63)
- no-connect marks 69 -> 127
Other:
- note added: "A"
- note added: "B"
- note added: "Backplane Connections"
- moved on the sheet: C?, JP5, JP7, R?, U1, U20B, U2B, U30A, U31A, U3C, U5A
